File: DecadeAmp.kicad_pcb (KiCad board)
At the start: 2 copper layers, 60 x 60 mm, 30 parts, among them J1 Conn_Coaxial, J2 Conn_Coaxial, SW1 SS-24E06-TG 5 (P), U1 MCP6V62-E/MS, U2 MCP6V62-E/MS

Commit message: Correct Op-Amp MCP6292-E/SN
Parts:
- U1, U2: value MCP6V62-E/MS -> MCP6292-E/SN
Changed lines of the file:
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@@
       (effects (font (size 1 1) (thickness 0.15)))
     )
-    (fp_text value MCP6V62-E/MS (at 0 3.5 270) (layer F.Fab)
+    (fp_text value MCP6292-E/SN (at 0 3.5 270) (layer F.Fab)
       (effects (font (size 1 1) (thickness 0.15)))
     )
@@
       (effects (font (size 1 1) (thickness 0.15)))
     )
-    (fp_text value MCP6V62-E/MS (at 0 3.5 270) (layer F.Fab)
+    (fp_text value MCP6292-E/SN (at 0 3.5 270) (layer F.Fab)
       (effects (font (size 1 1) (thickness 0.15)))
     )
