File: DecadeAmp.sch (KiCad schematic (older format))
At the start: 26 parts, among them J1 Conn_Coaxial, J2 Conn_Coaxial, SW1 SS-24E06-TG 5 (P), U1 MCP6V62-E/MS, U2 MCP6V62-E/MS

Commit message: Correct Op-Amp MCP6292-E/SN
Parts:
- U1, U2: value MCP6V62-E/MS -> MCP6292-E/SN
- gave numbers to parts that had none: 2
Changed lines of the file:
@@
 encoding utf-8
 Sheet 1 1
-Title ""
-Date ""
-Rev ""
-Comp ""
-Comment1 ""
+Title "Decade Amplifier"
+Date "2018-01-15"
+Rev "1.0.0"
+Comp "Ideas In Logic"
+Comment1 "© 2018 Wolfgang Jung"
 Comment2 ""
 Comment3 ""
@@
 P 2700 1750
 F 0 "U1" H 2700 1950 50  0000 L CNN
-F 1 "MCP6V62-E/MS" H 2700 1550 50  0000 L CNN
+F 1 "MCP6292-E/SN" H 2700 1550 50  0000 L CNN
 F 2 "Housings_SOIC:SOIC-8_3.9x4.9mm_Pitch1.27mm" H 2700 1750 50  0001 C CNN
 F 3 "" H 2700 1750 50  0001 C CNN
@@
 P 4100 1750
 F 0 "U1" H 4100 1950 50  0000 L CNN
-F 1 "MCP6V62-E/MS" H 4100 1550 50  0000 L CNN
+F 1 "MCP6292-E/SN" H 4100 1550 50  0000 L CNN
 F 2 "Housings_SOIC:SOIC-8_3.9x4.9mm_Pitch1.27mm" H 4100 1750 50  0001 C CNN
 F 3 "" H 4100 1750 50  0001 C CNN
@@
 P 5600 1750
 F 0 "U2" H 5600 1950 50  0000 L CNN
-F 1 "MCP6V62-E/MS" H 5600 1550 50  0000 L CNN
+F 1 "MCP6292-E/SN" H 5600 1550 50  0000 L CNN
 F 2 "Housings_SOIC:SOIC-8_3.9x4.9mm_Pitch1.27mm" H 5600 1750 50  0001 C CNN
 F 3 "" H 5600 1750 50  0001 C CNN
@@
 P 4100 4250
 F 0 "U2" H 4100 4450 50  0000 L CNN
-F 1 "MCP6V62-E/MS" H 4100 4050 50  0000 L CNN
+F 1 "MCP6292-E/SN" H 4100 4050 50  0000 L CNN
 F 2 "Housings_SOIC:SOIC-8_3.9x4.9mm_Pitch1.27mm" H 4100 4250 50  0001 C CNN
 F 3 "" H 4100 4250 50  0001 C CNN
@@
 $EndComp
 $Comp
-L GND #PWR01
+L GND #PWR2
 U 1 1 5A5D1D52
 P 1450 2200
-F 0 "#PWR01" H 1450 1950 50  0001 C CNN
+F 0 "#PWR2" H 1450 1950 50  0001 C CNN
 F 1 "GND" H 1450 2050 50  0000 C CNN
 F 2 "" H 1450 2200 50  0001 C CNN
@@
 Connection ~ 4000 1450
 $Comp
-L GND #PWR02
+L GND #PWR10
 U 1 1 5A5D1F3E
 P 5000 4250
-F 0 "#PWR02" H 5000 4000 50  0001 C CNN
+F 0 "#PWR10" H 5000 4000 50  0001 C CNN
 F 1 "GND" H 5000 4100 50  0000 C CNN
 F 2 "" H 5000 4250 50  0001 C CNN
@@
 Connection ~ 3550 4550
 $Comp
-L VEE #PWR03
+L VEE #PWR8
 U 1 1 5A5D2102
 P 3550 4400
-F 0 "#PWR03" H 3550 4250 50  0001 C CNN
+F 0 "#PWR8" H 3550 4250 50  0001 C CNN
 F 1 "VEE" H 3550 4550 50  0000 C CNN
 F 2 "" H 3550 4400 50  0001 C CNN
@@
 $EndComp
 $Comp
-L VCC #PWR04
+L VCC #PWR7
 U 1 1 5A5D214E
 P 3550 3750
-F 0 "#PWR04" H 3550 3600 50  0001 C CNN
+F 0 "#PWR7" H 3550 3600 50  0001 C CNN
 F 1 "VCC" H 3550 3900 50  0000 C CNN
 F 2 "" H 3550 3750 50  0001 C CNN
@@
 $EndComp
 $Comp
-L VCC #PWR05
+L VCC #PWR5
 U 1 1 5A5D224C
 P 3350 1450
-F 0 "#PWR05" H 3350 1300 50  0001 C CNN
+F 0 "#PWR5" H 3350 1300 50  0001 C CNN
 F 1 "VCC" H 3350 1600 50  0000 C CNN
 F 2 "" H 3350 1450 50  0001 C CNN
@@
 Connection ~ 4000 2050
 $Comp
-L VEE #PWR06
+L VEE #PWR6
 U 1 1 5A5D237D
 P 3500 2050
-F 0 "#PWR06" H 3500 1900 50  0001 C CNN
+F 0 "#PWR6" H 3500 1900 50  0001 C CNN
 F 1 "VEE" H 3500 2200 50  0000 C CNN
 F 2 "" H 3500 2050 50  0001 C CNN
@@
 $EndComp
 $Comp
-L GND #PWR07
+L GND #PWR4
 U 1 1 5A5D2A7B
 P 2150 2900
-F 0 "#PWR07" H 2150 2650 50  0001 C CNN
+F 0 "#PWR4" H 2150 2650 50  0001 C CNN
 F 1 "GND" H 2150 2750 50  0000 C CNN
 F 2 "" H 2150 2900 50  0001 C CNN
@@
 $EndComp
 $Comp
-L GND #PWR08
+L GND #PWR9
 U 1 1 5A5D2D1E
 P 3600 2900
-F 0 "#PWR08" H 3600 2650 50  0001 C CNN
+F 0 "#PWR9" H 3600 2650 50  0001 C CNN
 F 1 "GND" H 3600 2750 50  0000 C CNN
 F 2 "" H 3600 2900 50  0001 C CNN
@@
 $EndComp
 $Comp
-L GND #PWR09
+L GND #PWR11
 U 1 1 5A5D2DDB
 P 5050 2900
-F 0 "#PWR09" H 5050 2650 50  0001 C CNN
+F 0 "#PWR11" H 5050 2650 50  0001 C CNN
 F 1 "GND" H 5050 2750 50  0000 C CNN
 F 2 "" H 5050 2900 50  0001 C CNN
@@
 $EndComp
 $Comp
-L GND #PWR010
+L GND #PWR3
 U 1 1 5A5D405B
 P 1450 4600
-F 0 "#PWR010" H 1450 4350 50  0001 C CNN
+F 0 "#PWR3" H 1450 4350 50  0001 C CNN
 F 1 "GND" H 1450 4450 50  0000 C CNN
 F 2 "" H 1450 4600 50  0001 C CNN
@@
 	2800 3600 2600 3600
 $Comp
-L VEE #PWR011
+L VEE #PWR1
 U 1 1 5A5D36B4
 P 850 3900
-F 0 "#PWR011" H 850 3750 50  0001 C CNN
+F 0 "#PWR1" H 850 3750 50  0001 C CNN
 F 1 "VEE" H 850 4050 50  0000 C CNN
 F 2 "" H 850 3900 50  0001 C CNN
@@
 VMID
 $Comp
-L C C?
+L C C4
 U 1 1 5A5D4596
 P 5800 4000
-F 0 "C?" V 6050 3900 50  0000 L CNN
+F 0 "C4" V 6050 3900 50  0000 L CNN
 F 1 "100nF" V 5950 3900 50  0000 L CNN
 F 2 "Capacitors_SMD:C_0805" H 5838 3850 50  0001 C CNN
@@
 $EndComp
 $Comp
-L C C?
+L C C5
 U 1 1 5A5D4708
 P 6300 4000
-F 0 "C?" V 6550 3900 50  0000 L CNN
+F 0 "C5" V 6550 3900 50  0000 L CNN
 F 1 "100nF" V 6450 3900 50  0000 L CNN
 F 2 "Capacitors_SMD:C_0805" H 6338 3850 50  0001 C CNN
@@
 $EndComp
 $Comp
-L VEE #PWR?
+L VEE #PWR13
 U 1 1 5A5D4772
 P 5400 4150
-F 0 "#PWR?" H 5400 4000 50  0001 C CNN
+F 0 "#PWR13" H 5400 4000 50  0001 C CNN
 F 1 "VEE" H 5400 4300 50  0000 C CNN
 F 2 "" H 5400 4150 50  0001 C CNN
@@
 $EndComp
 $Comp
-L VCC #PWR?
+L VCC #PWR12
 U 1 1 5A5D47D1
 P 5400 3850
-F 0 "#PWR?" H 5400 3700 50  0001 C CNN
+F 0 "#PWR12" H 5400 3700 50  0001 C CNN
 F 1 "VCC" H 5400 4000 50  0000 C CNN
 F 2 "" H 5400 3850 50  0001 C CNN

Commit message: moved to new packages
Parts:
- C1, C2, C3, C4, C5: footprint Capacitors_SMD:C_0805 -> Capacitor_SMD:C_0805_2012Metric
- J1, J2: footprint Connectors:bnc-ci -> Connector_Coaxial:BNC_TEConnectivity_1478204_Vertical
- R1, R10, R11, R12, R13, R14, R15, R2, R3, R4, R5, R6, R7, R8, R9: footprint Resistors_SMD:R_0805 -> Resistor_SMD:R_0805_2012Metric
- U1, U2: footprint Housings_SOIC:SOIC-8_3.9x4.9mm_Pitch1.27mm -> Package_SOIC:SOIC-8_3.9x4.9mm_P1.27mm
Changed lines of the file:
@@
 Sheet 1 1
 Title "Decade Amplifier"
-Date "2018-01-15"
-Rev "1.0.0"
+Date "2018-01-26"
+Rev "1.0.1"
 Comp "Ideas In Logic"
 Comment1 "© 2018 Wolfgang Jung"
@@
 F 0 "U1" H 2700 1950 50  0000 L CNN
 F 1 "MCP6292-E/SN" H 2700 1550 50  0000 L CNN
-F 2 "Housings_SOIC:SOIC-8_3.9x4.9mm_Pitch1.27mm" H 2700 1750 50  0001 C CNN
+F 2 "Package_SOIC:SOIC-8_3.9x4.9mm_P1.27mm" H 2700 1750 50  0001 C CNN
 F 3 "" H 2700 1750 50  0001 C CNN
 	1    2700 1750
@@
 F 0 "U1" H 4100 1950 50  0000 L CNN
 F 1 "MCP6292-E/SN" H 4100 1550 50  0000 L CNN
-F 2 "Housings_SOIC:SOIC-8_3.9x4.9mm_Pitch1.27mm" H 4100 1750 50  0001 C CNN
+F 2 "Package_SOIC:SOIC-8_3.9x4.9mm_P1.27mm" H 4100 1750 50  0001 C CNN
 F 3 "" H 4100 1750 50  0001 C CNN
 	2    4100 1750
@@
 F 0 "U2" H 5600 1950 50  0000 L CNN
 F 1 "MCP6292-E/SN" H 5600 1550 50  0000 L CNN
-F 2 "Housings_SOIC:SOIC-8_3.9x4.9mm_Pitch1.27mm" H 5600 1750 50  0001 C CNN
+F 2 "Package_SOIC:SOIC-8_3.9x4.9mm_P1.27mm" H 5600 1750 50  0001 C CNN
 F 3 "" H 5600 1750 50  0001 C CNN
 	1    5600 1750
@@
 F 0 "U2" H 4100 4450 50  0000 L CNN
 F 1 "MCP6292-E/SN" H 4100 4050 50  0000 L CNN
-F 2 "Housings_SOIC:SOIC-8_3.9x4.9mm_Pitch1.27mm" H 4100 4250 50  0001 C CNN
+F 2 "Package_SOIC:SOIC-8_3.9x4.9mm_P1.27mm" H 4100 4250 50  0001 C CNN
 F 3 "" H 4100 4250 50  0001 C CNN
 	2    4100 4250
@@
 F 0 "J1" H 1460 1770 50  0000 C CNN
 F 1 "Conn_Coaxial" V 1565 1650 50  0000 C CNN
-F 2 "Connectors:bnc-ci" H 1450 1650 50  0001 C CNN
+F 2 "Connector_Coaxial:BNC_TEConnectivity_1478204_Vertical" H 1450 1650 50  0001 C CNN
 F 3 "" H 1450 1650 50  0001 C CNN
 	1    1450 1650
@@
 $EndComp
 $Comp
-L GND #PWR2
+L GND #PWR01
 U 1 1 5A5D1D52
 P 1450 2200
-F 0 "#PWR2" H 1450 1950 50  0001 C CNN
+F 0 "#PWR01" H 1450 1950 50  0001 C CNN
 F 1 "GND" H 1450 2050 50  0000 C CNN
 F 2 "" H 1450 2200 50  0001 C CNN
@@
 Connection ~ 4000 1450
 $Comp
-L GND #PWR10
+L GND #PWR02
 U 1 1 5A5D1F3E
 P 5000 4250
-F 0 "#PWR10" H 5000 4000 50  0001 C CNN
+F 0 "#PWR02" H 5000 4000 50  0001 C CNN
 F 1 "GND" H 5000 4100 50  0000 C CNN
 F 2 "" H 5000 4250 50  0001 C CNN
@@
 F 0 "R11" V 4680 4250 50  0000 C CNN
 F 1 "270" V 4600 4250 50  0000 C CNN
-F 2 "Resistors_SMD:R_0805" V 4530 4250 50  0001 C CNN
+F 2 "Resistor_SMD:R_0805_2012Metric" V 4530 4250 50  0001 C CNN
 F 3 "" H 4600 4250 50  0001 C CNN
 	1    4600 4250
@@
 F 0 "R6" V 3480 4400 50  0000 C CNN
 F 1 "100k" V 3400 4400 50  0000 C CNN
-F 2 "Resistors_SMD:R_0805" V 3330 4400 50  0001 C CNN
+F 2 "Resistor_SMD:R_0805_2012Metric" V 3330 4400 50  0001 C CNN
 F 3 "" H 3400 4400 50  0001 C CNN
 	1    3400 4400
@@
 F 0 "R5" V 3480 3900 50  0000 C CNN
 F 1 "100k" V 3400 3900 50  0000 C CNN
-F 2 "Resistors_SMD:R_0805" V 3330 3900 50  0001 C CNN
+F 2 "Resistor_SMD:R_0805_2012Metric" V 3330 3900 50  0001 C CNN
 F 3 "" H 3400 3900 50  0001 C CNN
 	1    3400 3900
@@
 Connection ~ 3550 4550
 $Comp
-L VEE #PWR8
+L VEE #PWR03
 U 1 1 5A5D2102
 P 3550 4400
-F 0 "#PWR8" H 3550 4250 50  0001 C CNN
+F 0 "#PWR03" H 3550 4250 50  0001 C CNN
 F 1 "VEE" H 3550 4550 50  0000 C CNN
 F 2 "" H 3550 4400 50  0001 C CNN
@@
 $EndComp
 $Comp
-L VCC #PWR7
+L VCC #PWR04
 U 1 1 5A5D214E
 P 3550 3750
-F 0 "#PWR7" H 3550 3600 50  0001 C CNN
+F 0 "#PWR04" H 3550 3600 50  0001 C CNN
 F 1 "VCC" H 3550 3900 50  0000 C CNN
 F 2 "" H 3550 3750 50  0001 C CNN
@@
 $EndComp
 $Comp
-L VCC #PWR5
+L VCC #PWR05
 U 1 1 5A5D224C
 P 3350 1450
-F 0 "#PWR5" H 3350 1300 50  0001 C CNN
+F 0 "#PWR05" H 3350 1300 50  0001 C CNN
 F 1 "VCC" H 3350 1600 50  0000 C CNN
 F 2 "" H 3350 1450 50  0001 C CNN
@@
 Connection ~ 4000 2050
 $Comp
-L VEE #PWR6
+L VEE #PWR06
 U 1 1 5A5D237D
 P 3500 2050
-F 0 "#PWR6" H 3500 1900 50  0001 C CNN
+F 0 "#PWR06" H 3500 1900 50  0001 C CNN
 F 1 "VEE" H 3500 2200 50  0000 C CNN
 F 2 "" H 3500 2050 50  0001 C CNN
@@
 F 0 "R4" V 3280 1750 50  0000 C CNN
 F 1 "270" V 3200 1750 50  0000 C CNN
-F 2 "Resistors_SMD:R_0805" V 3130 1750 50  0001 C CNN
+F 2 "Resistor_SMD:R_0805_2012Metric" V 3130 1750 50  0001 C CNN
 F 3 "" H 3200 1750 50  0001 C CNN
 	1    3200 1750
@@
 F 0 "R10" V 4680 1750 50  0000 C CNN
 F 1 "270" V 4600 1750 50  0000 C CNN
-F 2 "Resistors_SMD:R_0805" V 4530 1750 50  0001 C CNN
+F 2 "Resistor_SMD:R_0805_2012Metric" V 4530 1750 50  0001 C CNN
 F 3 "" H 4600 1750 50  0001 C CNN
 	1    4600 1750
@@
 F 0 "R15" V 6180 1750 50  0000 C CNN
 F 1 "270" V 6100 1750 50  0000 C CNN
-F 2 "Resistors_SMD:R_0805" V 6030 1750 50  0001 C CNN
+F 2 "Resistor_SMD:R_0805_2012Metric" V 6030 1750 50  0001 C CNN
 F 3 "" H 6100 1750 50  0001 C CNN
 	1    6100 1750
@@
 F 0 "R2" V 2530 2250 50  0000 C CNN
 F 1 "6k8" V 2450 2250 50  0000 C CNN
-F 2 "Resistors_SMD:R_0805" V 2380 2250 50  0001 C CNN
+F 2 "Resistor_SMD:R_0805_2012Metric" V 2380 2250 50  0001 C CNN
 F 3 "" H 2450 2250 50  0001 C CNN
 	1    2450 2250
@@
 F 0 "R3" V 2930 2250 50  0000 C CNN
 F 1 "2k2" V 2850 2250 50  0000 C CNN
-F 2 "Resistors_SMD:R_0805" V 2780 2250 50  0001 C CNN
+F 2 "Resistor_SMD:R_0805_2012Metric" V 2780 2250 50  0001 C CNN
 F 3 "" H 2850 2250 50  0001 C CNN
 	1    2850 2250
@@
 F 0 "R1" V 2230 2650 50  0000 C CNN
 F 1 "1k" V 2150 2650 50  0000 C CNN
-F 2 "Resistors_SMD:R_0805" V 2080 2650 50  0001 C CNN
+F 2 "Resistor_SMD:R_0805_2012Metric" V 2080 2650 50  0001 C CNN
 F 3 "" H 2150 2650 50  0001 C CNN
 	1    2150 2650
@@
 F 0 "C1" V 2900 2400 50  0000 L CNN
 F 1 "22pF" V 2800 2400 50  0000 L CNN
-F 2 "Capacitors_SMD:C_0805" H 2688 2350 50  0001 C CNN
+F 2 "Capacitor_SMD:C_0805_2012Metric" H 2688 2350 50  0001 C CNN
 F 3 "" H 2650 2500 50  0001 C CNN
 	1    2650 2500
@@
 $EndComp
 $Comp
-L GND #PWR4
+L GND #PWR07
 U 1 1 5A5D2A7B
 P 2150 2900
-F 0 "#PWR4" H 2150 2650 50  0001 C CNN
+F 0 "#PWR07" H 2150 2650 50  0001 C CNN
 F 1 "GND" H 2150 2750 50  0000 C CNN
 F 2 "" H 2150 2900 50  0001 C CNN
@@
 F 0 "R8" V 3930 2250 50  0000 C CNN
 F 1 "6k8" V 3850 2250 50  0000 C CNN
-F 2 "Resistors_SMD:R_0805" V 3780 2250 50  0001 C CNN
+F 2 "Resistor_SMD:R_0805_2012Metric" V 3780 2250 50  0001 C CNN
 F 3 "" H 3850 2250 50  0001 C CNN
 	1    3850 2250
@@
 F 0 "R9" V 4330 2250 50  0000 C CNN
 F 1 "2k2" V 4250 2250 50  0000 C CNN
-F 2 "Resistors_SMD:R_0805" V 4180 2250 50  0001 C CNN
+F 2 "Resistor_SMD:R_0805_2012Metric" V 4180 2250 50  0001 C CNN
 F 3 "" H 4250 2250 50  0001 C CNN
 	1    4250 2250
@@
 F 0 "R7" V 3680 2650 50  0000 C CNN
 F 1 "1k" V 3600 2650 50  0000 C CNN
-F 2 "Resistors_SMD:R_0805" V 3530 2650 50  0001 C CNN
+F 2 "Resistor_SMD:R_0805_2012Metric" V 3530 2650 50  0001 C CNN
 F 3 "" H 3600 2650 50  0001 C CNN
 	1    3600 2650
@@
 F 0 "C2" V 4300 2400 50  0000 L CNN
 F 1 "22pF" V 4200 2400 50  0000 L CNN
-F 2 "Capacitors_SMD:C_0805" H 4088 2350 50  0001 C CNN
+F 2 "Capacitor_SMD:C_0805_2012Metric" H 4088 2350 50  0001 C CNN
 F 3 "" H 4050 2500 50  0001 C CNN
 	1    4050 2500
@@
 $EndComp
 $Comp
-L GND #PWR9
+L GND #PWR08
 U 1 1 5A5D2D1E
 P 3600 2900
-F 0 "#PWR9" H 3600 2650 50  0001 C CNN
+F 0 "#PWR08" H 3600 2650 50  0001 C CNN
 F 1 "GND" H 3600 2750 50  0000 C CNN
 F 2 "" H 3600 2900 50  0001 C CNN
@@
 F 0 "R13" V 5430 2250 50  0000 C CNN
 F 1 "6k8" V 5350 2250 50  0000 C CNN
-F 2 "Resistors_SMD:R_0805" V 5280 2250 50  0001 C CNN
+F 2 "Resistor_SMD:R_0805_2012Metric" V 5280 2250 50  0001 C CNN
 F 3 "" H 5350 2250 50  0001 C CNN
 	1    5350 2250
@@
 F 0 "R14" V 5830 2250 50  0000 C CNN
 F 1 "2k2" V 5750 2250 50  0000 C CNN
-F 2 "Resistors_SMD:R_0805" V 5680 2250 50  0001 C CNN
+F 2 "Resistor_SMD:R_0805_2012Metric" V 5680 2250 50  0001 C CNN
 F 3 "" H 5750 2250 50  0001 C CNN
 	1    5750 2250
@@
 F 0 "R12" V 5130 2650 50  0000 C CNN
 F 1 "1k" V 5050 2650 50  0000 C CNN
-F 2 "Resistors_SMD:R_0805" V 4980 2650 50  0001 C CNN
+F 2 "Resistor_SMD:R_0805_2012Metric" V 4980 2650 50  0001 C CNN
 F 3 "" H 5050 2650 50  0001 C CNN
 	1    5050 2650
@@
 F 0 "C3" V 5800 2400 50  0000 L CNN
 F 1 "22pF" V 5700 2400 50  0000 L CNN
-F 2 "Capacitors_SMD:C_0805" H 5588 2350 50  0001 C CNN
+F 2 "Capacitor_SMD:C_0805_2012Metric" H 5588 2350 50  0001 C CNN
 F 3 "" H 5550 2500 50  0001 C CNN
 	1    5550 2500
@@
 $EndComp
 $Comp
-L GND #PWR11
+L GND #PWR09
 U 1 1 5A5D2DDB
 P 5050 2900
-F 0 "#PWR11" H 5050 2650 50  0001 C CNN
+F 0 "#PWR09" H 5050 2650 50  0001 C CNN
 F 1 "GND" H 5050 2750 50  0000 C CNN
 F 2 "" H 5050 2900 50  0001 C CNN
@@
 F 0 "J2" H 1460 4420 50  0000 C CNN
 F 1 "Conn_Coaxial" V 1565 4300 50  0000 C CNN
-F 2 "Connectors:bnc-ci" H 1450 4300 50  0001 C CNN
+F 2 "Connector_Coaxial:BNC_TEConnectivity_1478204_Vertical" H 1450 4300 50  0001 C CNN
 F 3 "" H 1450 4300 50  0001 C CNN
 	1    1450 4300
@@
 $EndComp
 $Comp
-L GND #PWR3
+L GND #PWR010
 U 1 1 5A5D405B
 P 1450 4600
-F 0 "#PWR3" H 1450 4350 50  0001 C CNN
+F 0 "#PWR010" H 1450 4350 50  0001 C CNN
 F 1 "GND" H 1450 4450 50  0000 C CNN
 F 2 "" H 1450 4600 50  0001 C CNN
@@
 	2800 3600 2600 3600
 $Comp
-L VEE #PWR1
+L VEE #PWR011
 U 1 1 5A5D36B4
 P 850 3900
-F 0 "#PWR1" H 850 3750 50  0001 C CNN
+F 0 "#PWR011" H 850 3750 50  0001 C CNN
 F 1 "VEE" H 850 4050 50  0000 C CNN
 F 2 "" H 850 3900 50  0001 C CNN
@@
 F 0 "C4" V 6050 3900 50  0000 L CNN
 F 1 "100nF" V 5950 3900 50  0000 L CNN
-F 2 "Capacitors_SMD:C_0805" H 5838 3850 50  0001 C CNN
+F 2 "Capacitor_SMD:C_0805_2012Metric" H 5838 3850 50  0001 C CNN
 F 3 "" H 5800 4000 50  0001 C CNN
 	1    5800 4000
@@
 F 0 "C5" V 6550 3900 50  0000 L CNN
 F 1 "100nF" V 6450 3900 50  0000 L CNN
-F 2 "Capacitors_SMD:C_0805" H 6338 3850 50  0001 C CNN
+F 2 "Capacitor_SMD:C_0805_2012Metric" H 6338 3850 50  0001 C CNN
 F 3 "" H 6300 4000 50  0001 C CNN
 	1    6300 4000
@@
 $EndComp
 $Comp
-L VEE #PWR13
+L VEE #PWR012
 U 1 1 5A5D4772
 P 5400 4150
-F 0 "#PWR13" H 5400 4000 50  0001 C CNN
+F 0 "#PWR012" H 5400 4000 50  0001 C CNN
 F 1 "VEE" H 5400 4300 50  0000 C CNN
 F 2 "" H 5400 4150 50  0001 C CNN
@@
 $EndComp
 $Comp
-L VCC #PWR12
+L VCC #PWR013
 U 1 1 5A5D47D1
 P 5400 3850
-F 0 "#PWR12" H 5400 3700 50  0001 C CNN
+F 0 "#PWR013" H 5400 3700 50  0001 C CNN
 F 1 "VCC" H 5400 4000 50  0000 C CNN
 F 2 "" H 5400 3850 50  0001 C CNN

Commit message: Better silkscreen, vendor-IDs of all components
Parts:
- BT1: Vendor (none) -> Keystone 1058
- C1, C2, C3: Vendor (none) -> 885012007002
- C4, C5: Vendor (none) -> C0805C104K5RACTU
- J1, J2: Vendor (none) -> TE-5-1634503-1
- R1, R12, R7: Vendor (none) -> RR1220P-102-D
- R10, R15, R4: Vendor (none) -> RC0805JR-07270RL
- R13, R2, R8: Vendor (none) -> RR1220P-682-D
- R14, R3, R9: Vendor (none) -> RR1220P-222-D
- R5, R6: Vendor (none) -> RR1220P-104-D
- SW1: Vendor (none) -> SS-24E06-TG 5 (P)
- U1: value MCP6292-E/SN -> MCP6V27-E/SN; Vendor (none) -> MCP6V27-E/SN
- U2: Vendor (none) -> MCP6292-E/SN
Changed lines of the file:
@@
 P 2700 1750
 F 0 "U1" H 2700 1950 50  0000 L CNN
-F 1 "MCP6292-E/SN" H 2700 1550 50  0000 L CNN
+F 1 "MCP6V27-E/SN" H 2700 1550 50  0000 L CNN
 F 2 "Package_SOIC:SOIC-8_3.9x4.9mm_P1.27mm" H 2700 1750 50  0001 C CNN
 F 3 "" H 2700 1750 50  0001 C CNN
+F 4 "MCP6V27-E/SN" H 2700 1750 60  0001 C CNN "Vendor"
 	1    2700 1750
 	1    0    0    -1
@@
 P 4100 1750
 F 0 "U1" H 4100 1950 50  0000 L CNN
-F 1 "MCP6292-E/SN" H 4100 1550 50  0000 L CNN
+F 1 "MCP6V27-E/SN" H 4100 1550 50  0000 L CNN
 F 2 "Package_SOIC:SOIC-8_3.9x4.9mm_P1.27mm" H 4100 1750 50  0001 C CNN
 F 3 "" H 4100 1750 50  0001 C CNN
+F 4 "MCP6V27-E/SN" H 4100 1750 60  0001 C CNN "Vendor"
 	2    4100 1750
 	1    0    0    -1
@@
 F 2 "Package_SOIC:SOIC-8_3.9x4.9mm_P1.27mm" H 5600 1750 50  0001 C CNN
 F 3 "" H 5600 1750 50  0001 C CNN
+F 4 "MCP6292-E/SN" H 5600 1750 60  0001 C CNN "Vendor"
 	1    5600 1750
 	1    0    0    -1
@@
 F 2 "Package_SOIC:SOIC-8_3.9x4.9mm_P1.27mm" H 4100 4250 50  0001 C CNN
 F 3 "" H 4100 4250 50  0001 C CNN
+F 4 "MCP6292-E/SN" H 4100 4250 60  0001 C CNN "Vendor"
 	2    4100 4250
 	1    0    0    -1
@@
 F 2 "SS-24E06-TG5:SS-24E06-TG 5 (P)" H 2000 4500 50  0001 C CNN
 F 3 "" H 2000 4500 50  0001 C CNN
+F 4 "SS-24E06-TG 5 (P)" H 2100 3900 60  0001 C CNN "Vendor"
 	1    2100 3900
 	1    0    0    -1
@@
 F 2 "Connector_Coaxial:BNC_TEConnectivity_1478204_Vertical" H 1450 1650 50  0001 C CNN
 F 3 "" H 1450 1650 50  0001 C CNN
+F 4 "TE-5-1634503-1" H 1450 1650 60  0001 C CNN "Vendor"
 	1    1450 1650
 	-1   0    0    -1
@@
 F 2 "Resistor_SMD:R_0805_2012Metric" V 3330 4400 50  0001 C CNN
 F 3 "" H 3400 4400 50  0001 C CNN
+F 4 "RR1220P-104-D" H 3400 4400 60  0001 C CNN "Vendor"
 	1    3400 4400
 	-1   0    0    1
@@
 F 2 "Resistor_SMD:R_0805_2012Metric" V 3330 3900 50  0001 C CNN
 F 3 "" H 3400 3900 50  0001 C CNN
+F 4 "RR1220P-104-D" H 3400 3900 60  0001 C CNN "Vendor"
 	1    3400 3900
 	-1   0    0    1
@@
 F 2 "Resistor_SMD:R_0805_2012Metric" V 3130 1750 50  0001 C CNN
 F 3 "" H 3200 1750 50  0001 C CNN
+F 4 "RC0805JR-07270RL" H 3200 1750 60  0001 C CNN "Vendor"
 	1    3200 1750
 	0    1    1    0
@@
 F 2 "Resistor_SMD:R_0805_2012Metric" V 4530 1750 50  0001 C CNN
 F 3 "" H 4600 1750 50  0001 C CNN
+F 4 "RC0805JR-07270RL" H 4600 1750 60  0001 C CNN "Vendor"
 	1    4600 1750
 	0    1    1    0
@@
 F 2 "Resistor_SMD:R_0805_2012Metric" V 6030 1750 50  0001 C CNN
 F 3 "" H 6100 1750 50  0001 C CNN
+F 4 "RC0805JR-07270RL" H 6100 1750 60  0001 C CNN "Vendor"
 	1    6100 1750
 	0    1    1    0
@@
 F 2 "Resistor_SMD:R_0805_2012Metric" V 2380 2250 50  0001 C CNN
 F 3 "" H 2450 2250 50  0001 C CNN
+F 4 "RR1220P-682-D" H 2450 2250 60  0001 C CNN "Vendor"
 	1    2450 2250
 	0    1    1    0
@@
 F 2 "Resistor_SMD:R_0805_2012Metric" V 2780 2250 50  0001 C CNN
 F 3 "" H 2850 2250 50  0001 C CNN
+F 4 "RR1220P-222-D" H 2850 2250 60  0001 C CNN "Vendor"
 	1    2850 2250
 	0    1    1    0
@@
 F 2 "Resistor_SMD:R_0805_2012Metric" V 2080 2650 50  0001 C CNN
 F 3 "" H 2150 2650 50  0001 C CNN
+F 4 "RR1220P-102-D" H 2150 2650 60  0001 C CNN "Vendor"
 	1    2150 2650
 	-1   0    0    1
@@
 F 2 "Capacitor_SMD:C_0805_2012Metric" H 2688 2350 50  0001 C CNN
 F 3 "" H 2650 2500 50  0001 C CNN
+F 4 "885012007002" H 2650 2500 60  0001 C CNN "Vendor"
 	1    2650 2500
 	0    1    1    0
@@
 F 2 "Resistor_SMD:R_0805_2012Metric" V 3780 2250 50  0001 C CNN
 F 3 "" H 3850 2250 50  0001 C CNN
+F 4 "RR1220P-682-D" H 3850 2250 60  0001 C CNN "Vendor"
 	1    3850 2250
 	0    1    1    0
@@
 F 2 "Resistor_SMD:R_0805_2012Metric" V 4180 2250 50  0001 C CNN
 F 3 "" H 4250 2250 50  0001 C CNN
+F 4 "RR1220P-222-D" H 4250 2250 60  0001 C CNN "Vendor"
 	1    4250 2250
 	0    1    1    0
@@
 F 2 "Resistor_SMD:R_0805_2012Metric" V 3530 2650 50  0001 C CNN
 F 3 "" H 3600 2650 50  0001 C CNN
+F 4 "RR1220P-102-D" H 3600 2650 60  0001 C CNN "Vendor"
 	1    3600 2650
 	-1   0    0    1
@@
 F 2 "Capacitor_SMD:C_0805_2012Metric" H 4088 2350 50  0001 C CNN
 F 3 "" H 4050 2500 50  0001 C CNN
+F 4 "885012007002" H 4050 2500 60  0001 C CNN "Vendor"
 	1    4050 2500
 	0    1    1    0
@@
 F 2 "Resistor_SMD:R_0805_2012Metric" V 5280 2250 50  0001 C CNN
 F 3 "" H 5350 2250 50  0001 C CNN
+F 4 "RR1220P-682-D" H 5350 2250 60  0001 C CNN "Vendor"
 	1    5350 2250
 	0    1    1    0
@@
 F 2 "Resistor_SMD:R_0805_2012Metric" V 5680 2250 50  0001 C CNN
 F 3 "" H 5750 2250 50  0001 C CNN
+F 4 "RR1220P-222-D" H 5750 2250 60  0001 C CNN "Vendor"
 	1    5750 2250
 	0    1    1    0
@@
 F 2 "Resistor_SMD:R_0805_2012Metric" V 4980 2650 50  0001 C CNN
 F 3 "" H 5050 2650 50  0001 C CNN
+F 4 "RR1220P-102-D" H 5050 2650 60  0001 C CNN "Vendor"
 	1    5050 2650
 	-1   0    0    1
@@
 F 2 "Capacitor_SMD:C_0805_2012Metric" H 5588 2350 50  0001 C CNN
 F 3 "" H 5550 2500 50  0001 C CNN
+F 4 "885012007002" H 5550 2500 60  0001 C CNN "Vendor"
 	1    5550 2500
 	0    1    1    0
@@
 F 2 "Battery_Holders:Keystone_1058_1x2032-CoinCell" V 1100 3860 50  0001 C CNN
 F 3 "" V 1100 3860 50  0001 C CNN
+F 4 "Keystone 1058" H 1100 3800 60  0001 C CNN "Vendor"
 	1    1100 3800
 	1    0    0    -1
@@
 F 2 "Connector_Coaxial:BNC_TEConnectivity_1478204_Vertical" H 1450 4300 50  0001 C CNN
 F 3 "" H 1450 4300 50  0001 C CNN
+F 4 "TE-5-1634503-1" H 1450 4300 60  0001 C CNN "Vendor"
 	1    1450 4300
 	-1   0    0    -1
@@
 F 2 "Capacitor_SMD:C_0805_2012Metric" H 5838 3850 50  0001 C CNN
 F 3 "" H 5800 4000 50  0001 C CNN
+F 4 "C0805C104K5RACTU" H 5800 4000 60  0001 C CNN "Vendor"
 	1    5800 4000
 	1    0    0    -1
@@
 F 2 "Capacitor_SMD:C_0805_2012Metric" H 6338 3850 50  0001 C CNN
 F 3 "" H 6300 4000 50  0001 C CNN
+F 4 "C0805C104K5RACTU" H 6300 4000 60  0001 C CNN "Vendor"
 	1    6300 4000
 	1    0    0    -1
